File: Graduation Cap Hardware/Graduation Cap/Graduation Cap.kicad_pcb (KiCad board)
At the start: 2 copper layers, 163.4 x 169.7 mm, 63 parts, among them IC1 ADXL335BCPZ-RL7, IC2 RP2040, J1 Conn_01x02, J2 USB_B_Micro, J3 Conn_01x04, J4 Conn_01x02, J5 Conn_01x03, U1 NCP1117-3.3_SOT223, U2 W25Q128JVS, Y1 ABM8-12.000MHz-20-B1U-T

Commit message: Updated pcb
Parts:
- removed the G*** at (87.9, 124.3)
- removed J1: Conn_01x02, Button_Switch_THT:SW_PUSH_6mm
- removed R4, R5: 27, Resistor_SMD:R_0201_0603Metric
- added G***: LOGO, UTEP_Logo_v1:utep_logo_v1, F.Cu at (125.6, 56.6)
- added SW1: SW_Push, Button_Switch_THT:SW_PUSH_6mm, F.Cu at (168.7, 78.9)
- moved J4 29.7 mm to (187.9, 116.5), turned to -45 degrees
- moved D17 24.2 mm to (193.2, 87.9), turned to -45 degrees
- moved J5 18.5 mm to (198.2, 109.5)
- moved R6 17.9 mm to (196.4, 91.0), turned to 135 degrees
- moved U1 9.69 mm to (181.9, 109.9), turned to 135 degrees
- moved C1 9.62 mm to (187.2, 107.4), turned to -45 degrees
- moved C2 8.75 mm to (184.3, 104.6), turned to -45 degrees
- moved C3 1.50 mm to (182.9, 95.6), turned to -90 degrees
Connections:
- IC2 pad 46: Net-(IC2-Pad46) -> /USB_D-
- IC2 pad 47: Net-(IC2-Pad47) -> /USB_D+
Routing:
- net +3V3: track 159.8 -> 170.0 mm, vias 9 -> 6
- net /USB_5V: track 13.5 -> 10.1 mm
- net Net-(IC2-Pad46): track 3.45 -> 0.00 mm
- net Net-(IC2-Pad47): track 3.25 -> 0.00 mm
- net +1V1: track 24.5 -> 27.5 mm
- net VBUS: track 13.3 -> 15.0 mm, vias 2 -> 0
- net /USB_D-: track 26.8 -> 27.8 mm
- net /USB_D+: track 27.1 -> 27.8 mm
- net /~USB_BOOT: track 24.0 -> 24.7 mm
- net /Bat: track 8.77 -> 8.18 mm
Other:
- board text added: "#GoMiners!"
- board text added: "JLCJLCJLCJLC"
- board text added: "Vbat"
- board text added: "Vbus"
- board text added: "Vusb"
