File: Graduation Cap Hardware/Graduation Cap/Graduation Cap.kicad_sch (KiCad schematic)
At the start: 59 parts, among them IC1 ADXL335BCPZ-RL7, IC2 RP2040, J1 Conn_01x02, J2 USB_B_Micro, J3 Conn_01x04, J4 Conn_01x02, J5 Conn_01x03, U1 NCP1117-3.3_SOT223, U2 W25Q128JVS, Y1 ABM8-12.000MHz-20-B1U-T

Commit message: Fix schematic
Other:
- note added: "05/14/2022"
- note removed: "03/18/2022"
Changed lines of the file:
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@@
     (effects (font (size 5 5)) (justify left bottom))
   )
-  (text "03/18/2022\n" (at 207.01 194.31 0)
+  (text "05/14/2022\n" (at 207.01 194.31 0)
     (effects (font (size 1.27 1.27)) (justify left bottom))
   )

Commit message: Updated pcb
Parts:
- removed J1: Conn_01x02, Button_Switch_THT:SW_PUSH_6mm, symbol Connector_Generic:Conn_01x02
- removed R4, R5: 27, Resistor_SMD:R_0201_0603Metric, symbol Device:R
- added SW1: SW_Push, Button_Switch_THT:SW_PUSH_6mm, symbol Switch:SW_Push
Connections:
- net GND: now also SW1.1
- net USB_D+: now also IC2.47 (USB_DP)
- net USB_D-: now also IC2.46 (USB_DM)
- net ~USB_BOOT: now also SW1.2
Other:
- note added: "Removed R3 and R4 to match USB impedance guidelines of 90 ohms"
- note removed: "Make sure R3 and R4 are close to RP2040"
Changed lines of the file:
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@@
+    (stroke (width 0) (type default) (color 0 0 0 0))
+  )
+  (wire (pts (xy 29.8196 95.25) (xy 31.6738 95.25))
     (stroke (width 0) (type default) (color 0 0 0 0))
   )
@@
     (stroke (width 0) (type default) (color 0 0 0 0))
   )
-  (wire (pts (xy 233.68 55.88) (xy 233.68 59.69))
+  (wire (pts (xy 233.68 55.88) (xy 233.68 73.66))
     (stroke (width 0) (type default) (color 0 0 0 0))
   )
@@
     (stroke (width 0) (type default) (color 0 0 0 0))
   )
-  (wire (pts (xy 41.91 95.25) (xy 53.594 95.25))
-    (stroke (width 0) (type default) (color 0 0 0 0))
-  )
   (wire (pts (xy 213.36 63.5) (xy 213.36 73.66))
     (stroke (width 0) (type default) (color 0 0 0 0))
@@
     (stroke (width 0) (type default) (color 0 0 0 0))
   )
-  (wire (pts (xy 44.45 99.06) (xy 44.45 97.79))
-    (stroke (width 0) (type default) (color 0 0 0 0))
-  )
   (polyline (pts (xy 187.96 163.83) (xy 284.48 163.83))
     (stroke (width 0) (type default) (color 0 0 0 0))
   )
-  (wire (pts (xy 231.14 55.88) (xy 231.14 59.69))
-    (stroke (width 0) (type default) (color 0 0 0 0))
-  )
   (polyline (pts (xy 121.92 163.449) (xy 121.92 167.005))
     (stroke (width 0) (type default) (color 0 0 0 0))
@@
     (stroke (width 0) (type default) (color 0 0 0 0))
   )
+  (wire (pts (xy 41.8338 95.25) (xy 53.594 95.25))
+    (stroke (width 0) (type default) (color 0 0 0 0))
+  )
   (wire (pts (xy 193.04 116.84) (xy 198.12 116.84))
     (stroke (width 0) (type default) (color 0 0 0 0))
@@
     (stroke (width 0) (type default) (color 0 0 0 0))
   )
-  (wire (pts (xy 233.68 67.31) (xy 233.68 73.66))
-    (stroke (width 0) (type default) (color 0 0 0 0))
-  )
   (wire (pts (xy 273.05 133.35) (xy 273.05 135.89))
     (stroke (width 0) (type default) (color 0 0 0 0))
@@
     (stroke (width 0) (type default) (color 0 0 0 0))
   )
-  (wire (pts (xy 44.45 97.79) (xy 41.91 97.79))
-    (stroke (width 0) (type default) (color 0 0 0 0))
-  )
   (polyline (pts (xy 120.65 123.19) (xy 184.15 123.19))
     (stroke (width 0) (type default) (color 0 0 0 0))
@@
     (stroke (width 0) (type default) (color 0 0 0 0))
   )
+  (wire (pts (xy 29.8196 96.5708) (xy 29.8196 95.25))
+    (stroke (width 0) (type default) (color 0 0 0 0))
+  )
   (polyline (pts (xy 115.57 149.86) (xy 20.32 149.86))
     (stroke (width 0) (type default) (color 0 0 0 0))
@@
     (stroke (width 0) (type default) (color 0 0 0 0))
   )
-  (wire (pts (xy 231.14 67.31) (xy 231.14 73.66))
+  (wire (pts (xy 231.14 55.88) (xy 231.14 73.66))
     (stroke (width 0) (type default) (color 0 0 0 0))
   )
@@
     (effects (font (size 1.27 1.27)) (justify right bottom))
   )
-  (text "Make sure R3 and R4 are close to RP2040\n" (at 236.22 59.69 0)
+  (text "Removed R3 and R4 to match USB \nimpedance guidelines of 90 ohms\n"
+    (at 235.9406 61.3664 0)
     (effects (font (size 1.27 1.27)) (justify left bottom))
   )
@@
     (effects (font (size 1.27 1.27)) (justify right bottom))
   )
-  (label "~USB_BOOT" (at 41.91 95.25 0)
+  (label "~USB_BOOT" (at 42.037 95.25 0)
     (effects (font (size 1.27 1.27)) (justify left bottom))
   )
@@
     )
     (pin "1")
+  )
+  (symbol (lib_id "Switch:SW_Push") (at 36.7538 95.25 0) (unit 1)
+    (in_bom yes) (on_board yes) (fields_autoplaced)
+    (property "Reference" "SW1" (id 0) (at 36.7538 86.5632 0))
+    (property "Value" "SW_Push" (id 1) (at 36.7538 89.1032 0))
+    (property "Footprint" "Button_Switch_THT:SW_PUSH_6mm" (id 2) (at 36.7538 90.17 0)
+      (effects (font (size 1.27 1.27)) hide)
+    )
+    (property "Datasheet" "~" (id 3) (at 36.7538 90.17 0)
+      (effects (font (size 1.27 1.27)) hide)
+    )
+    (pin "1")
+    (pin "2")
   )
   (symbol (lib_id "power:GND") (at 276.225 98.425 0) (unit 1)
@@
     (pin "1")
   )
-  (symbol (lib_id "Device:R") (at 233.68 63.5 0) (unit 1)
-    (in_bom yes) (on_board yes)
-    (property "Reference" "R5" (id 0) (at 234.95 62.23 0)
-      (effects (font (size 1.27 1.27)) (justify left))
-    )
-    (property "Value" "27" (id 1) (at 234.95 64.77 0)
-      (effects (font (size 1.27 1.27)) (justify left))
-    )
-    (property "Footprint" "Resistor_SMD:R_0201_0603Metric" (id 2) (at 231.902 63.5 90)
-      (effects (font (size 1.27 1.27)) hide)
-    )
-    (property "Datasheet" "~" (id 3) (at 233.68 63.5 0)
-      (effects (font (size 1.27 1.27)) hide)
-    )
-    (pin "1")
-    (pin "2")
-  )
   (symbol (lib_id "power:GND") (at 138.43 71.12 0) (unit 1)
     (in_bom yes) (on_board yes)
@@
     (pin "6")
   )
-  (symbol (lib_id "power:GND") (at 44.45 99.06 0) (unit 1)
-    (in_bom yes) (on_board yes) (fields_autoplaced)
-    (property "Reference" "#PWR04" (id 0) (at 44.45 105.41 0)
-      (effects (font (size 1.27 1.27)) hide)
-    )
-    (property "Value" "GND" (id 1) (at 44.45 104.14 0))
-    (property "Footprint" "" (id 2) (at 44.45 99.06 0)
-      (effects (font (size 1.27 1.27)) hide)
-    )
-    (property "Datasheet" "" (id 3) (at 44.45 99.06 0)
+  (symbol (lib_id "power:GND") (at 29.8196 96.5708 0) (unit 1)
+    (in_bom yes) (on_board yes) (fields_autoplaced)
+    (property "Reference" "#PWR04" (id 0) (at 29.8196 102.9208 0)
+      (effects (font (size 1.27 1.27)) hide)
+    )
+    (property "Value" "GND" (id 1) (at 29.8196 101.6508 0))
+    (property "Footprint" "" (id 2) (at 29.8196 96.5708 0)
+      (effects (font (size 1.27 1.27)) hide)
+    )
+    (property "Datasheet" "" (id 3) (at 29.8196 96.5708 0)
       (effects (font (size 1.27 1.27)) hide)
     )
@@
     )
     (pin "1")
-  )
-  (symbol (lib_id "Connector_Generic:Conn_01x02") (at 36.83 95.25 0) (mirror y) (unit 1)
-    (in_bom yes) (on_board yes) (fields_autoplaced)
-    (property "Reference" "J1" (id 0) (at 36.83 88.9 0))
-    (property "Value" "Conn_01x02" (id 1) (at 36.83 91.44 0))
-    (property "Footprint" "Button_Switch_THT:SW_PUSH_6mm" (id 2) (at 36.83 95.25 0)
-      (effects (font (size 1.27 1.27)) hide)
-    )
-    (property "Datasheet" "~" (id 3) (at 36.83 95.25 0)
-      (effects (font (size 1.27 1.27)) hide)
-    )
-    (pin "1")
-    (pin "2")
   )
   (symbol (lib_id "power:VBUS") (at 77.597 60.452 0) (unit 1)
@@
     (pin "1")
   )
-  (symbol (lib_id "Device:R") (at 231.14 63.5 0) (unit 1)
-    (in_bom yes) (on_board yes)
-    (property "Reference" "R4" (id 0) (at 227.33 62.23 0)
-      (effects (font (size 1.27 1.27)) (justify left))
-    )
-    (property "Value" "27" (id 1) (at 227.33 64.77 0)
-      (effects (font (size 1.27 1.27)) (justify left))
-    )
-    (property "Footprint" "Resistor_SMD:R_0201_0603Metric" (id 2) (at 229.362 63.5 90)
-      (effects (font (size 1.27 1.27)) hide)
-    )
-    (property "Datasheet" "~" (id 3) (at 231.14 63.5 0)
-      (effects (font (size 1.27 1.27)) hide)
-    )
-    (pin "1")
-    (pin "2")
-  )
   (symbol (lib_id "power:GND") (at 98.806 83.312 0) (unit 1)
     (in_bom yes) (on_board yes)
@@
       (reference "IC2") (unit 1) (value "RP2040") (footprint "RP2040 Pico:QFN40P700X700X90-57N-D")
     )
-    (path "/97327337-0f25-44a8-b23b-77126c7effa8"
-      (reference "J1") (unit 1) (value "Conn_01x02") (footprint "Button_Switch_THT:SW_PUSH_6mm")
-    )
     (path "/81596297-554a-4de2-8067-66e2218b2a33"
       (reference "J2") (unit 1) (value "USB_B_Micro") (footprint "Connector_USB:USB_Micro-B_Molex_47346-0001")
@@
       (reference "R3") (unit 1) (value "1k") (footprint "Resistor_SMD:R_0402_1005Metric")
     )
-    (path "/cbfcd6cb-7608-41a1-82b3-4f9b8e37b466"
-      (reference "R4") (unit 1) (value "27") (footprint "Resistor_SMD:R_0201_0603Metric")
-    )
-    (path "/5505ec85-32d3-4b02-8b4e-9f915802fada"
-      (reference "R5") (unit 1) (value "27") (footprint "Resistor_SMD:R_0201_0603Metric")
-    )
     (path "/7df46db5-2146-4bdc-8b7c-b247d64aedab"
       (reference "R6") (unit 1) (value "220") (footprint "Resistor_SMD:R_0603_1608Metric")
     )
+    (path "/3a92f55c-b0fd-4807-84bb-ec1b76146fd4"
+      (reference "SW1") (unit 1) (value "SW_Push") (footprint "Button_Switch_THT:SW_PUSH_6mm")
+    )
     (path "/b0b40da2-8918-4f0b-b11b-1408b929feb5"
